File: USB_SWD_PROGRAMMER/SWD_PROGRAMMER_minimal.sch (EAGLE design)
At the start: 19 parts

Commit message: Messing w/ Programmer
Tweaking USB
Parts:
- removed JP1: (no value), KW2:PINHD-2X5SMALL
- removed U$10: KW2_CPU_OFFSET, KW2:KW2_CPU_OFFSET
- removed U$3: KL20, KW2:KL20
- removed U$30: RA_BUTTON, KW2:RA_BUTTON
- removed U$46, U$59: 0.1uF, GW-devices:RF-C0805
- removed U$47, U$49, U$52: 10k, GW-devices:RF-R0805
- removed U$50, U$51: CJS, KW2:CJS
- removed U$62: 1uF, GW-devices:RF-C0805
- removed U$63: 10uF, GW-devices:RF-C0805
- removed U$64: CSTCE8M00G55-R0, KW2:CSTCE8M00G55-R0
- added C1: 10uF, GW-devices:RF-C0805
- added C2: 1uF, GW-devices:RF-C0805
- added C3, C4: 0.1uF, GW-devices:RF-C0805
- added JP3: (no value), pinhead:PINHD-1X11
- added R1, R3, R4, R5, R6: 10k, GW-devices:RF-R0805
- added R2: 5k, GW-devices:RF-R0805
- added S1: RA_BUTTON, KW2:RA_BUTTON
- added U$1: KL20_48, KW2:KL20_48
- added X1: CSTCE8M00G55-R0, KW2:CSTCE8M00G55-R0
- renumbered U$13 to D2, U$14 to J1, U$9 to D1
Connections:
- removed net N$35: D1.2, J1.D-, U$3.USB0_DM
- removed net N$36: D2.2, J1.D+, U$3.USB0_DP
- removed net N$52: JP2.2, U$3.PTA3, U$47.2
- removed net N$55: JP2.4, U$3.PTA0
- removed net N$56: JP2.6, U$3.PTA2
- removed net N$57: JP2.8, U$3.PTA1
- removed net N$58: JP2.10, U$3.RST, U$49.2
- removed net SWD_CLK: JP1.4, U$10.PTA0/JTAG_TCLK/SWD_CLK/EZP_CLK/!UART0_CTS/!UART0_COL/FTM0_CH5, U$51.P$1
- removed net SWD_DIO: JP1.2, U$10.PTA3/JTAG_TMS/SWD_DIO/UART0_RTS/FTM0_CH0, U$50.P$1
- removed net SWD_TGT_CLK: U$3.PTC5, U$51.P$2
- new net CLK: JP2.4, U$1.PTA0
- new net D_N: D1.2, J1.D-, R5.1
- new net D_P: D2.2, J1.D+, R4.1
- new net JRST: JP2.10, JP3.8, R2.2, R6.1, U$1.RESET_B
- new net N$3: JP3.4, U$1.VBAT
- new net N$7: JP3.5, U$1.VOUT33
- new net N$8: JP3.6, U$1.VREGIN
- new net N$9: R5.2, U$1.USB0_DM
- new net TDI: JP2.8, U$1.PTA1
- new net TDO: JP2.6, U$1.PTA2
- new net TMS: JP2.2, R3.2, U$1.PTA3
- net +3V3: now also C1.2, C2.2, C3.2, C4.2, JP3.10, JP3.11, JP3.9, R1.1, R3.1, U$1.VDD, U$1.VDD1, U$1.VDDA; no longer JP1.1, U$10.+3V3@1, U$10.+3V3@2, U$3.VDD, U$3.VDDA, U$3.VOUT33, U$46.2, U$47.1, U$49.1, U$52.1, U$59.2, U$62.2, U$63.2
- net GND: now also C1.1, C2.1, C3.1, C4.1, JP3.1, JP3.2, JP3.3, R6.2, S1.1, U$1.VSS, U$1.VSS1, U$1.VSSA, X1.2; no longer JP1.3, JP1.5, U$10.GND@1, U$10.GND@2, U$10.GND@3, U$10.GND@4, U$3.VSS, U$3.VSSA, U$30.1, U$46.1, U$59.1, U$62.1, U$63.1, U$64.2
- net N$1: now also R4.2, U$1.USB0_DP; no longer U$3.PTC6, U$3.PTC7, U$50.P$2
- net N$2: now also JP3.7, R2.1; no longer U$3.VREGIN
- net N$4: now also U$1.PTA18, X1.1; no longer U$3.PTA18, U$64.1
- net N$6: now also U$1.PTA19, X1.3; no longer U$3.PTA19, U$64.3
- net RST: now also R1.2, S1.2, U$1.PTB1; no longer JP1.10, U$10.!RESET, U$3.PTB1, U$30.2, U$52.2
Other:
- moved on the sheet: JP2
